Commit message: Made some progress

File: nuturtle_description/urdf/common_properties.xacro (robot description, xacro)
@@ -2,4 +2,7 @@
 <robot name="xacro_properties" xmlns:xacro="http://ros.org/wiki/xacro">
   <!-- Init colour -->
+  <material name="purple">
+    <color rgba="0.3 0.16 0.52 1.0"/>
+  </material>
   <material name="black">
       <color rgba="0.0 0.0 0.0 1.0"/>

File: nuturtle_description/urdf/turtlebot3_burger.urdf.xacro (robot description, xacro)
@@ -8,4 +8,5 @@
   <xacro:property name="TRACK_WIDTH" value="${params['track_width']}" />
   <xacro:property name="COLLISION_RADIUS" value="${params['collision_radius']}" />
+  <xacro:arg name="color" default="purple"/>
   <link name="base_footprint"/>
   <joint name="base_joint" type="fixed">
@@ -20,5 +21,5 @@
         <mesh filename="package://nuturtle_description/meshes/burger_base.stl" scale="0.001 0.001 0.001"/>
       </geometry>
-      <material name="light_black"/>
+      <material name="$(arg color)"/>
     </visual>
     <collision>
